File: kagisys_shield.kicad_pcb (KiCad board)
At the start: 2 copper layers, 6 parts, among them J1 Conn1, J2 Conn_01x04_Female, J3 Conn_01x03_Female, J4 Conn_01x02_Female, J5 Conn_01x02_Female, J6 Conn_01x04_Female

Commit message: fix pcb
Parts:
- added Q1: Q_NMOS_GSD, Package_TO_SOT_SMD:SOT-23, F.Cu at (124.6, 80.5)
- added Q2: Q_NMOS_GSD, Package_TO_SOT_SMD:SOT-23, F.Cu at (131.8, 84.2)
- added R1: 10k, Resistor_THT:R_Axial_DIN0309_L9.0mm_D3.2mm_P12.70mm_Horizontal, F.Cu at (104.5, 80.5)
- added R2: 10k, Resistor_THT:R_Axial_DIN0309_L9.0mm_D3.2mm_P12.70mm_Horizontal, F.Cu at (104.5, 86.5)
- J1: footprint Connector_PinHeader_2.54mm:PinHeader_2x06_P2.54mm_Horizontal -> Connector_PinHeader_2.54mm:PinHeader_2x07_P2.54mm_Horizontal
- moved J3 69.3 mm to (108.2, 99.0)
- moved J1 53.9 mm to (104.8, 56.8)
- moved J4 40.7 mm to (125.5, 99.0)
- moved J2 35.5 mm to (140.0, 99.0), turned to 90 degrees
- moved J6 31.5 mm to (159.0, 99.0), turned to 90 degrees
- moved J5 15.1 mm to (179.2, 99.0), turned to 90 degrees
Connections:
- J1 pad 10: GPIO0_B7 -> GND
- J1 pad 11: GND -> GPIO2_A2
- J1 pad 12: GPIO0_C0 -> GPIO0_B7
- J1 pad 2: GPIO0_B3 -> 3.3V
- J1 pad 3: GND -> 5V
- J1 pad 4: GPIO0_B4 -> GPIO0_B3
- J1 pad 5: GPIO2_A1 -> GND
- J1 pad 6: GPIO2_A5 -> GPIO0_B4
- J1 pad 7: GPIO2_A0 -> GPIO2_A1
- J1 pad 8: GND -> GPIO2_A5
- J1 pad 9: GPIO2_A2 -> GPIO2_A0
- J3 pad 1: GND -> Net-(J3-Pad1)
- J3 pad 3: GPIO0_B7 -> Net-(J3-Pad3)
- J5 pad 1: 5V -> 3.3V
Routing:
- net 3.3V: track 0.00 -> 132.6 mm, vias 0 -> 1
- net GPIO2_A0: track 43.3 -> 105.0 mm, vias 0 -> 1
- net GPIO0_B3: track 17.4 -> 60.9 mm
- net GPIO2_A2: track 0.00 -> 42.4 mm
- net GPIO0_B4: track 21.0 -> 58.2 mm
- net 5V: track 103.0 -> 139.8 mm
- net Net-(J3-Pad1): track 0.00 -> 36.0 mm, vias 0 -> 1
- net Net-(J3-Pad3): track 0.00 -> 35.5 mm, vias 0 -> 1
- net GND: track 105.1 -> 137.0 mm, vias 0 -> 1
- net GPIO0_C0: track 20.6 -> 40.5 mm
- net GPIO0_B7: track 34.5 -> 21.3 mm
- net GPIO2_A5: track 72.2 -> 83.7 mm
- net GPIO2_A1: track 83.8 -> 90.0 mm, vias 0 -> 1
Other:
- net class Default: trace_width 0.25 -> 0.5
